Commit message: feat: add inertial properties to xacro and configure gitignore

File: src/my_robot_description/urdf/common_properties.xacro (robot description, xacro)
@@ -1,9 +1,37 @@
 <?xml version="1.0"?>
 <robot xmlns:xacro="http://www.ros.org/wiki/xacro">
-        <material name="green">
-            <color rgba="0 0.6 0 1"/>
-        </material>
-        <material name="gray">
-            <color rgba="0.7 0.7 0.7 1"/>
-        </material>
+    <material name="green">
+        <color rgba="0 0.6 0 1"/>
+    </material>
+    <material name="gray">
+        <color rgba="0.7 0.7 0.7 1"/>
+    </material>
+    <!-- Macro for the box inertia -->
+    <xacro:macro name="box_inertia" params="m x y z o_xyz o_rpy">
+        <inertial>
+            <origin xyz="${o_xyz}" rpy="${o_rpy}"/>
+            <mass value="${m}"/>
+            <inertia ixx="${(1/12)*m * (y*y + z*z)}" ixy="0" ixz="0"
+                iyy="${(1/12)*m * (x*x + z*z)}" iyz="0"
+                izz="${(1/12)*m * (y*y + x*x)}"/>
+        </inertial>
+    </xacro:macro>
+    <!-- Macro for the cylinder inertia -->
+    <xacro:macro name="cylinder_inertia" params="m r l o_xyz o_rpy">
+        <inertial>
+            <origin xyz="${o_xyz}" rpy="${o_rpy}"/>
+            <mass value="${m}"/>
+            <inertia ixx="${(1/12)*m * (3*r*r + l*l)}" ixy="0" ixz="0"
+                iyy="${(1/12)*m * (3*r*r + l*l)}" iyz="0"
+                izz="${(1/2)*m*r*r}"/>
+        </inertial>
+    </xacro:macro>
+    <!-- Macro for the sphere inertia -->
+    <xacro:macro name="sphere_inertia" params="m r o_xyz o_rpy">
+        <inertial>
+            <origin xyz="${o_xyz}" rpy="${o_rpy}"/>
+            <mass value="${m}"/>
+            <inertia ixx="${(2/5)*m*r*r}" ixy="0" ixz="0" iyy="${(2/5)*m*r*r}" iyz="0" izz="${(2/5)*m*r*r}"/>
+        </inertial>
+    </xacro:macro>
 </robot>

File: src/my_robot_description/urdf/mobile_base.xacro (robot description, xacro)
@@ -17,4 +17,6 @@
                     <material name="gray"/>
                 </visual>
+                <!-- Inertial property -->
+                <xacro:cylinder_inertia m="1.0" r="${wheel_radius}" l="${wheel_length}" o_xyz="0 0 0" o_rpy="${pi/2} 0 0"/>
             </link>
         </xacro:macro>
@@ -28,4 +30,6 @@
                 <material name="green"/>
             </visual>
+            <!-- Inertial property -->
+            <xacro:box_inertia m="5.0" x="${base_length}" y="${base_width}" z="${base_height}" o_xyz="0 0 ${base_height/2.0}" o_rpy="0 0 0"/>
         </link>
         <!-- Right wheel link -->
@@ -58,4 +62,6 @@
                 <origin xyz="0 0 0" rpy="0 0 0"/>
             </visual>
+            <!-- Inertial property -->
+            <xacro:sphere_inertia m="0.5" r="${wheel_radius/2.0}" o_xyz="0 0 0" o_rpy="0 0 0"/>
         </link>
         <!-- Caster wheel and base joint -->
